File: hardware/attinier84-motherboard-mk-3.0.sch (EAGLE design)
At the start: 8 parts, among them IC1 ATTINY84, U1 ATTINIER84_SHIELD1551GSMD

Commit message: finished up motherboard, initial shield dicking
Parts:
- RESET: value SPST-NO-TACT3MM-PTH-SMALL-PADS -> SPST-NO-TACT3MM-RA; device A_butts:SPST-NO-TACT3MM-PTH-SMALL-PADS -> A_butts:SPST-NO-TACT3MM-RA
Connections:
- net N$1: now also BATT.+1; no longer BATT.+
Changed lines of the file:
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@@
 <setting verticaltext="up"/>
 </settings>
-<grid distance="100" unitdist="mil" unit="mil" style="lines" multiple="1" display="yes" altdistance="2" altunitdist="mil" altunit="mil"/>
+<grid distance="100" unitdist="mil" unit="mil" style="lines" multiple="1" display="yes" altdistance="1" altunitdist="mil" altunit="mil"/>
 <layers>
 <layer number="1" name="Top" color="4" fill="1" visible="yes" active="no"/>
@@
 <schematic xreflabel="%F%N/%S.%C%R" xrefpart="/%S.%C%R">
 <attributes>
+<attribute name="REVISION" value="3.0"/>
 </attributes>
 <variantdefs>
@@
 </classes>
 <parts>
-<part name="FRAME1" library="A_butts" deviceset="FRAME-LETTER" device="NO_PACKAGE"/>
+<part name="FRAME1" library="A_butts" deviceset="FRAME-LETTER" device="NO_PACKAGE">
+<attribute name="VERSION" value=""/>
+</part>
 <part name="BATT" library="A_butts" deviceset="BATTERY-COIN" device="CR2032_SMD" value="CR2032"/>
 <part name="IC1" library="A_butts" deviceset="ATTINY84" device=""/>
@@
 <part name="SUPPLY2" library="A_butts" deviceset="VCC" device=""/>
 <part name="SUPPLY3" library="A_butts" deviceset="VCC" device=""/>
-<part name="RESET" library="A_butts" deviceset="SPST-NO-TACT" device="3MM-PTH-SMALL-PADS" value="SPST-NO-TACT3MM-PTH-SMALL-PADS"/>
+<part name="RESET" library="A_butts" deviceset="SPST-NO-TACT" device="3MM-RA" value="SPST-NO-TACT3MM-RA"/>
 <part name="GND3" library="A_butts" deviceset="GND" device=""/>
 <part name="U1" library="A_butts" deviceset="ATTINIER84_SHIELD" device="1551GSMD" value="ATTINIER84_SHIELD1551GSMD"/>
@@
 <net name="N$1" class="0">
 <segment>
-<pinref part="BATT" gate="G$1" pin="+"/>
-<wire x1="50.8" y1="43.18" x2="50.8" y2="45.72" width="0.1524" layer="91"/>
 <pinref part="PWR" gate="G$1" pin="COM"/>
-<wire x1="50.8" y1="45.72" x2="55.88" y2="45.72" width="0.1524" layer="91"/>
-</segment>
-</net>
+<wire x1="48.26" y1="45.72" x2="55.88" y2="45.72" width="0.1524" layer="91"/>
+<pinref part="BATT" gate="G$1" pin="+1"/>
+<wire x1="48.26" y1="40.64" x2="48.26" y2="45.72" width="0.1524" layer="91"/>
+</segment>
+</net>
