File: hardware/attinier84-2digit-shield-mk-2.0.sch (EAGLE design)
At the start: 5 parts, among them IC1 TMP36, U1 ATTINIER84_SHIELD1551G

Commit message: temp shield with display done
Parts:
- removed C1: 0.1uF, A_butts:CAPACITOR-CERAMIC025-024X044
- DISPLAY1: value 7SEG_2DIG19MM -> 7SEG_2DIG14MM; device A_butts:7SEG_2DIG19MM -> A_butts:7SEG_2DIG14MM
Connections:
- net GND: no longer C1.2
- net PA0: now also IC1.VCC; no longer DISPLAY1.C
- net PA1: now also IC1.OUT; no longer DISPLAY1.DP
- net PA2: now also DISPLAY1.DIG1; no longer DISPLAY1.E
- net PA3: now also DISPLAY1.A; no longer DISPLAY1.D
- net PA4: now also DISPLAY1.B; no longer DISPLAY1.DIG1
- net PA5: now also DISPLAY1.G; no longer DISPLAY1.B
- net PA6: now also DISPLAY1.C; no longer DISPLAY1.A
- net PA7: now also DISPLAY1.DIG2; no longer IC1.OUT
- net PB0: now also DISPLAY1.E; no longer DISPLAY1.G
- net PB1: now also DISPLAY1.F; no longer DISPLAY1.DIG2
- net PB2: now also DISPLAY1.D; no longer DISPLAY1.F
- net VCC: no longer C1.1, IC1.VCC
Other:
- moved on the sheet: DISPLAY1
